Commit message: added nav2

File: install/articubot_one/share/articubot_one/description/org_robot_core.xacro (robot description, xacro)
@@ -2,4 +2,18 @@
 <robot xmlns:xacro="http://www.ros.org/wiki/xacro" >
     <xacro:include filename="inertial_macros.xacro"/>
+    <xacro:property name="chassis_length" value="0.335"/>
+    <xacro:property name="chassis_width" value="0.265"/>
+    <xacro:property name="chassis_height" value="0.138"/>
+    <xacro:property name="chassis_mass" value="1.0"/>
+    <xacro:property name="wheel_radius" value="0.033"/>
+    <xacro:property name="wheel_thickness" value="0.026"/>
+    <xacro:property name="wheel_mass" value="0.05"/>
+    <xacro:property name="wheel_offset_x" value="0.226"/>
+    <xacro:property name="wheel_offset_y" value="0.1485"/>
+    <xacro:property name="wheel_offset_z" value="0.01"/>
+    <xacro:property name="caster_wheel_radius" value="0.01"/>
+    <xacro:property name="caster_wheel_mass" value="0.01"/>
+    <xacro:property name="caster_wheel_offset_x" value="0.075"/>
+    <xacro:property name="caster_wheel_offset_z" value="${wheel_offset_z - wheel_radius + caster_wheel_radius}"/>
     <material name="white">
         <color rgba="1 1 1 1" />
@@ -14,6 +28,17 @@
         <color rgba="0 0 0 1"/>
     </material>
+    <material name="red">
+        <color rgba="1 0 0 1"/>
+    </material>
     <!-- BASE LINK -->
     <link name="base_link">
+    </link>
+    <!-- BASE_FOOTPRINT LINK -->
+    <joint name="base_footprint_joint" type="fixed">
+        <parent link="base_link"/>
+        <child link="base_footprint"/>
+        <origin xyz="0 0 0" rpy="0 0 0"/>
+    </joint>
+    <link name="base_footprint">
     </link>
     <!-- CHASSIS LINK -->
@@ -21,26 +46,26 @@
         <parent link="base_link"/>
         <child link="chassis"/>
-        <origin xyz="-0.1 0 0"/>
+        <origin xyz="${-wheel_offset_x} 0 ${-wheel_offset_z}"/>
     </joint>
     <link name="chassis">
         <visual>
-            <origin xyz="0.15 0 0.075"/>
+            <origin xyz="${chassis_length/2} 0 ${chassis_height/2}"/>
             <geometry>
-                <box size="0.3 0.3 0.15"/>
+                <box size="${chassis_length} ${chassis_width} ${chassis_height}"/>
             </geometry>
-            <material name="white"/>
+            <material name="orange"/>
         </visual>
         <collision>
-            <origin xyz="0.15 0 0.075"/>
+            <origin xyz="${chassis_length/2} 0 ${chassis_height/2}"/>
             <geometry>
-                <box size="0.3 0.3 0.15"/>
+                <box size="${chassis_length} ${chassis_width} ${chassis_height}"/>
             </geometry>
         </collision>
-        <xacro:inertial_box mass="0.5" x="0.3" y="0.3" z="0.15">
-            <origin xyz="0.15 0 0.075" rpy="0 0 0"/>
+        <xacro:inertial_box mass="0.5" x="${chassis_length}" y="${chassis_width}" z="${chassis_height}">
+            <origin xyz="${chassis_length/2} 0 ${chassis_height/2}" rpy="0 0 0"/>
         </xacro:inertial_box>
     </link>
     <gazebo reference="chassis">
-        <material>Gazebo/White</material>
+        <material>Gazebo/Orange</material>
     </gazebo>
     <!-- LEFT WHEEL LINK -->
@@ -48,5 +73,5 @@
         <parent link="base_link"/>
         <child link="left_wheel"/>
-        <origin xyz="0 0.175 0" rpy="-${pi/2} 0 0" />
+        <origin xyz="0 ${wheel_offset_y} 0" rpy="-${pi/2} 0 0" />
         <axis xyz="0 0 1"/>
     </joint>
@@ -54,5 +79,5 @@
         <visual>
             <geometry>
-                <cylinder radius="0.05" length="0.04"/>
+                <cylinder radius="${wheel_radius}" length="${wheel_thickness}"/>
             </geometry>
             <material name="blue"/>
@@ -60,8 +85,8 @@
         <collision>
             <geometry>
-                <cylinder radius="0.05" length="0.04"/>
+                <sphere radius="${wheel_radius}"/>
             </geometry>
         </collision>
-        <xacro:inertial_cylinder mass="0.1" length="0.04" radius="0.05">
+        <xacro:inertial_cylinder mass="${wheel_mass}" length="${wheel_thickness}" radius="${wheel_radius}">
             <origin xyz="0 0 0" rpy="0 0 0"/>
         </xacro:inertial_cylinder>
@@ -74,5 +99,5 @@
         <parent link="base_link"/>
         <child link="right_wheel"/>
-        <origin xyz="0 -0.175 0" rpy="${pi/2} 0 0" />
+        <origin xyz="0 ${-wheel_offset_y} 0" rpy="${pi/2} 0 0" />
         <axis xyz="0 0 -1"/>
     </joint>
@@ -80,5 +105,5 @@
         <visual>
             <geometry>
-                <cylinder radius="0.05" length="0.04"/>
+                <cylinder radius="${wheel_radius}" length="${wheel_thickness}"/>
             </geometry>
             <material name="blue"/>
@@ -86,8 +111,8 @@
         <collision>
             <geometry>
-                <cylinder radius="0.05" length="0.04"/>
+                <sphere radius="${wheel_radius}"/>
             </geometry>
         </collision>
-        <xacro:inertial_cylinder mass="0.1" length="0.04" radius="0.05">
+        <xacro:inertial_cylinder mass="${wheel_mass}" length="${wheel_thickness}" radius="${wheel_radius}">
             <origin xyz="0 0 0" rpy="0 0 0"/>
         </xacro:inertial_cylinder>
@@ -100,257 +125,26 @@
         <parent link="chassis"/>
         <child link="caster_wheel"/>
-        <origin xyz="0.24 0 0"/>
+        <origin xyz="${caster_wheel_offset_x} 0 ${caster_wheel_offset_z}"/>
     </joint>
     <link name="caster_wheel">
         <visual>
             <geometry>
-                <sphere radius="0.05"/>
+                <sphere radius="${caster_wheel_radius}"/>
             </geometry>
-            <material name="black"/>
+            <material name="white"/>
         </visual>
         <collision>
             <geometry>
-                <sphere radius="0.05"/>
+                <sphere radius="${caster_wheel_radius}"/>
             </geometry>
         </collision>
-        <xacro:inertial_sphere mass="0.1" radius="0.05">
+        <xacro:inertial_sphere mass="${caster_wheel_mass}" radius="${caster_wheel_radius}">
             <origin xyz="0 0 0" rpy="0 0 0"/>
         </xacro:inertial_sphere>
     </link>
     <gazebo reference="caster_wheel">
-        <material>Gazebo/Black</material>
+        <material>Gazebo/White</material>
         <mu1 value="0.001"/>
         <mu2 value="0.001"/>
     </gazebo>
 </robot>
-<!-- <?xml version="1.0"?>
-<robot xmlns:xacro="http://www.ros.org/wiki/xacro" >
-    <xacro:include filename="inertial_macros.xacro"/>
-    <material name="white">
-        <color rgba="1 1 1 1" />
-    </material>
-    <material name="orange">
-        <color rgba="1 0.3 0.1 1"/>
-    </material>
-    <material name="blue">
-        <color rgba="0.2 0.2 1 1"/>
-    </material>
-    <material name="black">
-        <color rgba="0 0 0 1"/>
-    </material>
-    <!-- BASE LINK -->
-    <link name="world">
-    </link>
-    <link name="base_link">
-        <parent link="world"/>
-        <child link="base_link"/>
-        <origin xyz="0 0 0"/>
-    </link>
-    <!-- CHASSIS LINK -->
-    <joint name="chassis_joint" type="fixed">
-        <parent link="base_link"/>
-        <child link="chassis"/>
-        <origin xyz="-0.1 0 0"/>
-    </joint>
-    <link name="chassis">
-        <visual>
-            <origin xyz="0.15 0 0.075"/>
-            <geometry>
-                <box size="0.3 0.3 0.15"/>
-            </geometry>
-            <material name="white"/>
-        </visual>
-        <collision>
-            <origin xyz="0.15 0 0.075"/>
-            <geometry>
-                <box size="0.3 0.3 0.15"/>
-            </geometry>
-        </collision>
-        <xacro:inertial_box mass="0.5" x="0.3" y="0.3" z="0.15">
-            <origin xyz="0.15 0 0.075" rpy="0 0 0"/>
-        </xacro:inertial_box>
-    </link>
-    <gazebo reference="chassis">
-        <material>Gazebo/White</material>
-    </gazebo>
-    <!-- LEFT WHEEL LINK -->
-    <joint name="left_wheel_joint" type="continuous">
-        <parent link="base_link"/>
-        <child link="left_wheel"/>
-        <origin xyz="0 0.175 0" rpy="-${pi/2} 0 0" />
-        <axis xyz="0 0 1"/>
-    </joint>
-    <link name="left_wheel">
-        <visual>
-            <geometry>
-                <cylinder radius="0.05" length="0.04"/>
-            </geometry>
-            <material name="blue"/>
-        </visual>
-        <collision>
-            <geometry>
-                <cylinder radius="0.05" length="0.04"/>
-            </geometry>
-        </collision>
-        <xacro:inertial_cylinder mass="0.1" length="0.04" radius="0.05">
-            <origin xyz="0 0 0" rpy="0 0 0"/>
-        </xacro:inertial_cylinder>
-    </link>
-    <gazebo reference="left_wheel">
-        <material>Gazebo/Blue</material>
-    </gazebo>
-    <!-- RIGHT WHEEL LINK -->
-    <joint name="right_wheel_joint" type="continuous">
-        <parent link="base_link"/>
-        <child link="right_wheel"/>
-        <origin xyz="0 -0.175 0" rpy="${pi/2} 0 0" />
-        <axis xyz="0 0 -1"/>
-    </joint>
-    <link name="right_wheel">
-        <visual>
-            <geometry>
-                <cylinder radius="0.05" length="0.04"/>
-            </geometry>
-            <material name="blue"/>
-        </visual>
-        <collision>
-            <geometry>
-                <cylinder radius="0.05" length="0.04"/>
-            </geometry>
-        </collision>
-        <xacro:inertial_cylinder mass="0.1" length="0.04" radius="0.05">
-            <origin xyz="0 0 0" rpy="0 0 0"/>
-        </xacro:inertial_cylinder>
-    </link>
-    <gazebo reference="right_wheel">
-        <material>Gazebo/Blue</material>
-    </gazebo>
-    <!-- CASTER WHEEL LINK -->
-    <joint name="caster_wheel_joint" type="fixed">
-        <parent link="chassis"/>
-        <child link="caster_wheel"/>
-        <origin xyz="0.24 0 0"/>
-    </joint>
-    <link name="caster_wheel">
-        <visual>
-            <geometry>
-                <sphere radius="0.05"/>
-            </geometry>
-            <material name="black"/>
-        </visual>
-        <collision>
-            <geometry>
-                <sphere radius="0.05"/>
-            </geometry>
-        </collision>
-        <xacro:inertial_sphere mass="0.1" radius="0.05">
-            <origin xyz="0 0 0" rpy="0 0 0"/>
-        </xacro:inertial_sphere>
-    </link>
-    <gazebo reference="caster_wheel">
-        <material>Gazebo/Black</material>
-        <mu1 value="0.001"/>
-        <mu2 value="0.001"/>
-    </gazebo>
-    <!-- Define the static obstacle link -->
-    <link name="obstacle_box">
-        <visual>
-            <origin xyz="5 2 2" rpy="0 0 0"/> <!-- Position of the obstacle -->
-            <geometry>
-                <box size="2 2 2"/> <!-- Size of the obstacle -->
-            </geometry>
-            <material name="black"/> <!-- Color of the obstacle -->
-        </visual>
-        <collision>
-            <origin xyz="5 2 2" rpy="0 0 0"/> <!-- Position of the obstacle -->
-            <geometry>
-                <box size="2 2 2"/> <!-- Size of the obstacle -->
-            </geometry>
-        </collision>
-    </link>
-    <!-- Define a static joint to keep the box fixed in place -->
-    <joint name="obstacle_joint" type="fixed">
-        <parent link="world"/> <!-- Attach it to the world frame -->
-        <child link="obstacle_box"/>
-        <origin xyz="5 2 2" rpy="0 0 0"/> <!-- Position of the obstacle -->
-    </joint>
-    <!-- Optionally add the obstacle to the Gazebo simulation -->
-    <gazebo reference="obstacle_box">
-        <material>Gazebo/Orange</material>
-    </gazebo>
-</robot> -->
-<!--
-     <!-- Main Actuator Link (Single Entity) -->
-    <link name="actuator_main_link">
-        <inertial>
-            <mass value="4.0"/>
-            <origin xyz="0 0 0"/>
-            <inertia ixx="0.2" iyy="0.2" izz="0.2" ixy="0" ixz="0" iyz="0"/>
-        </inertial>
-    </link>
-    <!-- Prismatic Joint (Moves the Actuator as One Unit) -->
-    <joint name="linear_actuator" type="prismatic">
-        <parent link="base_link"/>
-        <child link="actuator_main_link"/>
-        <origin xyz="0.35 0 0" rpy="0 -${pi/2} 0"/>
-        <axis xyz="1 0 0"/>  <!-- Moves in X-direction -->
-        <limit lower="0" upper="0.5" effort="10.0" velocity="0.5"/>
-    </joint>
-    <!-- Actuator Link 1 (Fixed to Main Actuator) -->
-    <link name="actuator_link">
-        <inertial>
-            <mass value="2.0"/>
-            <origin xyz="0 0 0"/>
-            <inertia ixx="0.1" iyy="0.1" izz="0.1" ixy="0" ixz="0" iyz="0"/>
-        </inertial>
-        <visual>
-            <geometry>
-                <box size="0.01 0.08 0.3"/>
-            </geometry>
-        </visual>
-        <collision>
-            <geometry>
-                <box size="0.01 0.08 0.3"/>
-            </geometry>
-        </collision>
-        <xacro:inertial_box mass="2.0" x="0.01" y="0.08" z="0.3">
-            <origin xyz="0 0 0" rpy="0 0 0"/>
-        </xacro:inertial_box>
-    </link>
-    <joint name="fixed_actuator1" type="fixed">
-        <parent link="actuator_main_link"/>
-        <child link="actuator_link"/>
-        <origin xyz="0 0.075 0"/>
-    </joint>
-    <gazebo reference="fixed_actuator1">
-        <material>Gazebo/Blue</material>
-    </gazebo>
-    <!-- Actuator Link 2 (Fixed to Main Actuator) -->
-    <link name="actuator_link2">
-        <inertial>
-            <mass value="2.0"/>
-            <origin xyz="0 0 0"/>
-            <inertia ixx="0.1" iyy="0.1" izz="0.1" ixy="0" ixz="0" iyz="0"/>
-        </inertial>
-        <visual>
-            <geometry>
-                <box size="0.01 0.08 0.3"/>
-            </geometry>
-        </visual>
-        <collision>
-            <geometry>
-                <box size="0.01 0.08 0.3"/>
-            </geometry>
-        </collision>
-        <xacro:inertial_box mass="2.0" x="0.01" y="0.08" z="0.3">
-            <origin xyz="0 0 0" rpy="0 0 0"/>
-        </xacro:inertial_box>
-    </link>
-    <joint name="fixed_actuator2" type="fixed">
-        <parent link="actuator_main_link"/>
-        <child link="actuator_link2"/>
-        <origin xyz="0 -0.075 0"/>
-    </joint>
-    <gazebo reference="fixed_actuator2">
-        <material>Gazebo/Blue</material>
-    </gazebo> -->
