Commit message: added goal position publisher and removed rotaiion deviation

File: install/articubot_one/share/articubot_one/description/robot_core.xacro (robot description, xacro)
@@ -125,5 +125,5 @@
             </geometry>
         </collision>
-        <xacro:inertial_sphere mass="5" radius="0.05">
+        <xacro:inertial_sphere mass="2" radius="0.05">
             <origin xyz="0 0 0" rpy="0 0 0"/>
         </xacro:inertial_sphere>
@@ -136,5 +136,5 @@
     <link name="actuator_main_link">
         <inertial>
-            <mass value="0.4"/>
+            <mass value="0.0002"/>
             <origin xyz="0 0 0"/>
             <inertia ixx="0.2" iyy="0.2" izz="0.2" ixy="0" ixz="0" iyz="0"/>
@@ -152,5 +152,5 @@
     <link name="actuator_link">
         <inertial>
-            <mass value="0.2"/>
+            <mass value="0.0001"/>
             <origin xyz="0 0 0"/>
             <inertia ixx="0.1" iyy="0.1" izz="0.1" ixy="0" ixz="0" iyz="0"/>
@@ -166,5 +166,5 @@
             </geometry>
         </collision>
-        <xacro:inertial_box mass="0.2" x="0.5" y="0.08" z="0.01">
+        <xacro:inertial_box mass="0.0001" x="0.5" y="0.08" z="0.01">
             <origin xyz="0 0 0" rpy="0 0 0"/>
         </xacro:inertial_box>
@@ -181,5 +181,5 @@
     <link name="actuator_link2">
         <inertial>
-            <mass value="0.2"/>
+            <mass value="0.0001"/>
             <origin xyz="0 0 0"/>
             <inertia ixx="0.1" iyy="0.1" izz="0.1" ixy="0" ixz="0" iyz="0"/>
@@ -195,5 +195,5 @@
             </geometry>
         </collision>
-        <xacro:inertial_box mass="0.2" x="0.5" y="0.08" z="0.01">
+        <xacro:inertial_box mass="0.0001" x="0.5" y="0.08" z="0.01">
             <origin xyz="0 0 0" rpy="0 0 0"/>
         </xacro:inertial_box>
